Commit message: Stage 2.1 Use RL to enable random target following

File: assets_own/mobile_manipulator_little_xy_link.urdf (robot description, URDF)
Before this commit: robot Robot, 12 links, 11 joints
Links:
- link base_link_x: mass 1.00000000 -> 0.0100000000
- link base_link_y: mass 1.00000000 -> 0.0100000000
Joints:
- joint joint_theta: child base_link_x -> abstract_chassis_link; limit lower=-3.14159265 upper=3.14159265 effort=100.0 velocity=2.5 -> lower=-Inf upper=Inf effort=100.0 velocity=2.5; parent base -> base_link_y
- joint joint_x: child base_link_y -> base_link_x; parent base_link_x -> base
- joint joint_y: child abstract_chassis_link -> base_link_y; parent base_link_y -> base_link_x
