Commit message: feat: validate semantic RS4 riser playback

File: assets_own/recomoProto2_two_wheel_riser/recomoProto2_two_wheel_riser.urdf (robot description, URDF)
Before this commit: robot recomoProto2-two-wheel-riser, 14 links, 13 joints
Joints:
- joint camera_optical_center: origin xyz=0 0.0065609 0.10147 rpy=0 -1.5708 0 -> xyz=0 0.0065609 0.10147 rpy=3.141592653573 -1.570792653590 -1.570796326778
- joint joint1_gimbal_pitch: axis 0 0 1 -> 1.000000000000 0.000000000000 -0.000000000000; limit lower=-3.2 upper=1.57 effort=10.0 velocity=0.5 -> effort=10.0 velocity=6.283185307180; type revolute -> continuous
- joint joint2_gimbal_roll: axis 0 0 1 -> 0.000000000000 1.000000000000 0.000000000000; limit lower=-3.2 upper=1.57 effort=10.0 velocity=0.5 -> lower=-1.658062789395 upper=4.188790204786 effort=10.0 velocity=6.283185307180
- joint joint3_gimbal_yaw: limit lower=-3.1416 upper=3.1416 effort=10.0 velocity=0.5 -> lower=-1.954768762234 upper=3.735004599268 effort=10.0 velocity=6.283185307180; origin xyz=0.000003410742927 0.147436171819393 0 rpy=1.5708 0 0 -> xyz=-0.071543364669 0.131332738755 0.034914221454 rpy=-1.750353420000 1.408789120000 -2.995696870000
